Commit message: Done Section 4: Locomotion

File: bumperbot_ws/install/bumperbot_description/share/bumperbot_description/urdf/bumperbot.urdf.xacro (robot description, xacro)
@@ -1,142 +1 @@
-<?xml version="1.0"?>
-<robot name="bumperbot" xmlns:xacro="http://ros.org/wiki/xacro">
-  <!-- Include Gazebo Parameters -->
-  <xacro:include filename="$(find bumperbot_description)/urdf/bumperbot_gazebo.xacro" />
-  <!-- Links -->
-  <link name="base_footprint"/>
-  <link name="base_link">
-    <visual>
-      <origin xyz="0 0 0" rpy="0 0 0" />
-      <geometry>
-        <mesh filename="package://bumperbot_description/meshes/base_link.STL" />
-      </geometry>
-    </visual>
-    <collision>
-      <origin xyz="0 0 0" rpy="0 0 0" />
-      <geometry>
-        <mesh filename="package://bumperbot_description/meshes/base_link.STL" />
-      </geometry>
-    </collision>
-    <inertial>
-      <origin xyz="0 0 0.04" rpy="0.0 0.25 0.3" />
-      <mass value="8.2573504e-01"/>
-      <inertia ixx="2.2124416e-02" ixy="-1.2294101e-04" ixz="3.4938785e-04"
-                                   iyy="2.1193702e-02"  iyz="-5.0120904e-05"
-                                                        izz="2.0064271e-02" />
-    </inertial>
-  </link>
-  <link name="wheel_right_link">
-    <visual>
-      <origin xyz="0 0 0" rpy="1.57 0 0" />
-      <geometry>
-        <mesh filename="package://bumperbot_description/meshes/wheel_right_link.STL" />
-      </geometry>
-    </visual>
-    <collision>
-      <origin xyz="0 -0.015 0" rpy="1.57 0 0" />
-      <geometry>
-        <sphere radius="0.033"/>
-      </geometry>
-    </collision>
-    <inertial>
-      <origin xyz="0 -0.014 0" rpy="0 0 0" />
-      <mass value="0.0530086090966721" />
-      <inertia ixx="1.88176298336665E-05" ixy="-4.8444933029987E-10" ixz="1.88163708851143E-08"
-                                          iyy="3.11510738647764E-05" iyz="-6.93560663069607E-11"
-                                                                     izz="1.8801969558182E-05" />
-    </inertial>
-  </link>
-  <link name="wheel_left_link">
-    <visual>
-      <origin xyz="0 0 0" rpy="-1.57 0 0" />
-      <geometry>
-        <mesh filename="package://bumperbot_description/meshes/wheel_left_link.STL" />
-      </geometry>
-    </visual>
-    <collision>
-      <origin xyz="0 0.015 0" rpy="-1.57 0 0" />
-      <geometry>
-        <sphere radius="0.033"/>
-      </geometry>
-    </collision>
-    <inertial>
-      <origin xyz="0 0.014 0" rpy="0 0 0" />
-      <mass value="0.0530086043217644" />
-      <inertia ixx="1.8792911368909E-05"  ixy="3.31256392204584E-10" ixz="-1.14082001662767E-08"
-                                          iyy="3.11510738759073E-05" iyz="-3.60499245082192E-10"
-                                                                     izz="1.88266886146847E-05" />
-    </inertial>
-  </link>
-  <link name="caster_front_link">
-    <visual>
-      <origin xyz="0 0 0" rpy="0 0 0" />
-      <geometry>
-        <mesh filename="package://bumperbot_description/meshes/caster_front_link.STL" />
-      </geometry>
-    </visual>
-    <collision>
-      <origin xyz="0 0 0" rpy="0 0 0" />
-      <geometry>
-        <sphere radius="0.005"/>
-      </geometry>
-    </collision>
-    <inertial>
-      <origin xyz="3.89968128948481E-07 2.40073004698083E-07 0.00219173397061506" rpy="0 0 0" />
-      <mass value="1.44379265037903E-06" />
-      <inertia ixx="7.23075276010246E-11" ixy="-6.10956883467859E-16" ixz="2.22849693525031E-15"
-                                          iyy="3.8713793085917E-11"   iyz="2.93909858781952E-15"
-                                                                      izz="1.00967486676306E-10" />
-    </inertial>
-  </link>
-  <link name="caster_rear_link">
-    <visual>
-      <origin xyz="0 0 0" rpy="0 0 0" />
-      <geometry>
-        <mesh filename="package://bumperbot_description/meshes/caster_rear_link.STL" />
-      </geometry>
-    </visual>
-    <collision>
-      <origin xyz="0 0 0" rpy="0 0 0" />
-      <geometry>
-        <sphere radius="0.005"/>
-      </geometry>
-    </collision>
-    <inertial>
-      <origin xyz="3.8996812895542E-07 2.40073004698083E-07 0.00219173397061509" rpy="0 0 0" />
-      <mass value="1.44379265037902E-06" />
-      <inertia ixx="7.23075276010246E-11" ixy="-6.10956872363424E-16" ixz="2.22849693527207E-15"
-                                          iyy="3.87137930859167E-11"  iyz="2.939098587861E-15"
-                                                                      izz="1.00967486676306E-10" />
-    </inertial>
-  </link>
-  <!-- Joints -->
-  <joint name="base_joint" type="fixed">
-    <parent link="base_footprint"/>
-    <child link="base_link" />
-    <origin xyz="0 0 0.033" rpy="0 0 0"/>
-  </joint>
-  <joint name="wheel_right_joint" type="continuous">
-    <origin xyz="0 -0.0701101849418637 0" rpy="0 0 0" />
-    <parent link="base_link" />
-    <child link="wheel_right_link" />
-    <axis xyz="0 1 0" />
-  </joint>
-  <joint name="wheel_left_joint" type="continuous">
-    <origin xyz="0 0.0701101849418642 0" rpy="0 0 0" />
-    <parent link="base_link" />
-    <child link="wheel_left_link" />
-    <axis xyz="0 1 0" />
-  </joint>
-  <joint name="caster_front_joint" type="fixed">
-    <origin xyz="0.04755 0 -0.0275" rpy="0 0 0" />
-    <parent link="base_link" />
-    <child link="caster_front_link" />
-    <axis xyz="0 0 0" />
-  </joint>
-  <joint name="caster_rear_joint" type="fixed">
-    <origin xyz="-0.04755 0 -0.0275" rpy="0 0 0" />
-    <parent link="base_link" />
-    <child link="caster_rear_link" />
-    <axis xyz="0 0 0" />
-  </joint>
-</robot>
+/home/raz/projects/self_driving_OC_project/bumperbot_ws/src/bumperbot_description/urdf/bumperbot.urdf.xacro

File: bumperbot_ws/install/bumperbot_description/share/bumperbot_description/urdf/bumperbot_gazebo.xacro (robot description, xacro)
@@ -1,39 +1 @@
-<?xml version="1.0"?>
-<robot name="bumperbot" xmlns:xacro="http://ros.org/wiki/xacro">
-  <!-- Wheels -->
-  <gazebo reference="wheel_left_link">
-    <mu1>1000000000000000.0</mu1>
-    <mu2>1000000000000000.0</mu2>
-    <kp>1000000000000.0</kp>
-    <kd>10.0</kd>
-    <minDepth>0.001</minDepth>
-    <maxVel>0.1</maxVel>
-    <fdir1>1 0 0</fdir1>
-  </gazebo>
-  <gazebo reference="wheel_right_link">
-    <mu1>1000000000000000.0</mu1>
-    <mu2>1000000000000000.0</mu2>
-    <kp>1000000000000.0</kp>
-    <kd>10.0</kd>
-    <minDepth>0.001</minDepth>
-    <maxVel>0.1</maxVel>
-    <fdir1>1 0 0</fdir1>
-  </gazebo>
-  <!-- Caster Wheels -->
-  <gazebo reference="caster_rear_link">
-    <mu1>0.1</mu1>
-    <mu2>0.1</mu2>
-    <kp>1000000.0</kp>
-    <kd>100.0</kd>
-    <minDepth>0.001</minDepth>
-    <maxVel>1.0</maxVel>
-  </gazebo>
-  <gazebo reference="caster_front_link">
-    <mu1>0.1</mu1>
-    <mu2>0.1</mu2>
-    <kp>1000000.0</kp>
-    <kd>100.0</kd>
-    <minDepth>0.001</minDepth>
-    <maxVel>1.0</maxVel>
-  </gazebo>
-</robot>
+/home/raz/projects/self_driving_OC_project/bumperbot_ws/src/bumperbot_description/urdf/bumperbot_gazebo.xacro

File: bumperbot_ws/src/bumperbot_description/urdf/bumperbot.urdf.xacro (robot description, xacro)
@@ -1,20 +1,29 @@
 <?xml version="1.0"?>
 <robot name="bumperbot" xmlns:xacro="http://ros.org/wiki/xacro">
+  <!-- Include Common Properties -->
+  <xacro:include filename="$(find bumperbot_description)/urdf/common_properties.xacro" />
   <!-- Include Gazebo Parameters -->
   <xacro:include filename="$(find bumperbot_description)/urdf/bumperbot_gazebo.xacro" />
+  <!-- Useful XACRO Variables (Properties) -->
+  <xacro:property name="effort" value="30.0" />
+  <xacro:property name="velocity" value="10.0" />
+  <!-- Dimensions -->
+  <xacro:property name="wheel_length" value="0.03" />
+  <xacro:property name="wheel_radius" value="0.033" />
   <!-- Links -->
   <link name="base_footprint"/>
   <link name="base_link">
     <visual>
-      <origin xyz="0 0 0" rpy="0 0 0" />
       <geometry>
         <mesh filename="package://bumperbot_description/meshes/base_link.STL" />
       </geometry>
+      <origin xyz="0 0 0" rpy="0 0 0" />
+      <material name="green" />
     </visual>
     <collision>
-      <origin xyz="0 0 0" rpy="0 0 0" />
       <geometry>
         <mesh filename="package://bumperbot_description/meshes/base_link.STL" />
       </geometry>
+      <origin xyz="0 0 0" rpy="0 0 0" />
     </collision>
     <inertial>
@@ -28,14 +37,15 @@
   <link name="wheel_right_link">
     <visual>
-      <origin xyz="0 0 0" rpy="1.57 0 0" />
       <geometry>
         <mesh filename="package://bumperbot_description/meshes/wheel_right_link.STL" />
       </geometry>
+      <origin xyz="0 0 0" rpy="1.57 0 0" />
+      <material name="black" />
     </visual>
     <collision>
-      <origin xyz="0 -0.015 0" rpy="1.57 0 0" />
       <geometry>
-        <sphere radius="0.033"/>
+        <sphere radius="${wheel_radius}"/>
       </geometry>
+      <origin xyz="0 -${wheel_length / 2.0} 0" rpy="1.57 0 0" />
     </collision>
     <inertial>
@@ -49,14 +59,15 @@
   <link name="wheel_left_link">
     <visual>
-      <origin xyz="0 0 0" rpy="-1.57 0 0" />
       <geometry>
         <mesh filename="package://bumperbot_description/meshes/wheel_left_link.STL" />
       </geometry>
+      <origin xyz="0 0 0" rpy="-1.57 0 0" />
+      <material name="black" />
     </visual>
     <collision>
-      <origin xyz="0 0.015 0" rpy="-1.57 0 0" />
       <geometry>
-        <sphere radius="0.033"/>
+        <sphere radius="${wheel_radius}"/>
       </geometry>
+      <origin xyz="0 ${wheel_length / 2.0} 0" rpy="-1.57 0 0" />
     </collision>
     <inertial>
@@ -70,14 +81,15 @@
   <link name="caster_front_link">
     <visual>
-      <origin xyz="0 0 0" rpy="0 0 0" />
       <geometry>
         <mesh filename="package://bumperbot_description/meshes/caster_front_link.STL" />
       </geometry>
+      <material name="white" />
     </visual>
+      <origin xyz="0 0 0" rpy="0 0 0" />
     <collision>
-      <origin xyz="0 0 0" rpy="0 0 0" />
       <geometry>
         <sphere radius="0.005"/>
       </geometry>
+      <origin xyz="0 0 0" rpy="0 0 0" />
     </collision>
     <inertial>
@@ -91,14 +103,15 @@
   <link name="caster_rear_link">
     <visual>
-      <origin xyz="0 0 0" rpy="0 0 0" />
       <geometry>
         <mesh filename="package://bumperbot_description/meshes/caster_rear_link.STL" />
       </geometry>
+      <origin xyz="0 0 0" rpy="0 0 0" />
+      <material name="white" />
     </visual>
     <collision>
-      <origin xyz="0 0 0" rpy="0 0 0" />
       <geometry>
         <sphere radius="0.005"/>
       </geometry>
+      <origin xyz="0 0 0" rpy="0 0 0" />
     </collision>
     <inertial>
@@ -110,4 +123,19 @@
     </inertial>
   </link>
+  <!-- <link name="can_link">
+    <visual>
+      <geometry>
+        <mesh filename="package://bumperbot_description/meshes/can.STL" />
+      </geometry>
+      <origin xyz="-0.0325 0.0325 0" rpy="1.57 0 0" />
+      <material name="red" />
+    </visual>
+    <collision>
+      <geometry>
+        <mesh filename="package://bumperbot_description/meshes/can.STL" />
+      </geometry>
+      <origin xyz="-0.0325 0.0325 0" rpy="1.57 0 0" />
+    </collision>
+  </link> -->
   <!-- Joints -->
   <joint name="base_joint" type="fixed">
@@ -140,3 +168,9 @@
     <axis xyz="0 0 0" />
   </joint>
+  <!-- <joint name="can_joint" type="fixed">
+    <origin xyz="0 0 0.078" rpy="0 0 0" />
+    <parent link="base_link" />
+    <child link="can_link" />
+    <axis xyz="0 0 0" />
+  </joint> -->
 </robot>

File: bumperbot_ws/src/bumperbot_description/urdf/bumperbot_gazebo.xacro (robot description, xacro)
@@ -1,4 +1,15 @@
 <?xml version="1.0"?>
 <robot name="bumperbot" xmlns:xacro="http://ros.org/wiki/xacro">
+  <!-- Base -->
+  <gazebo reference="base_link">
+    <visual>
+      <material>
+        <ambient>0 1 0 1</ambient>
+        <diffuse>0 1 0 1</diffuse>
+        <specular>0.1 0.1 0.1 1</specular>
+      </material>
+    </visual>
+    <!-- Green -->
+  </gazebo>
   <!-- Wheels -->
   <gazebo reference="wheel_left_link">
@@ -10,4 +21,12 @@
     <maxVel>0.1</maxVel>
     <fdir1>1 0 0</fdir1>
+    <visual>
+      <material>
+        <ambient>0 0 0 1</ambient>
+        <diffuse>0 0 0 1</diffuse>
+        <specular>0.1 0.1 0.1 1</specular>
+      </material>
+    </visual>
+    <!-- Black -->
   </gazebo>
   <gazebo reference="wheel_right_link">
@@ -19,4 +38,12 @@
     <maxVel>0.1</maxVel>
     <fdir1>1 0 0</fdir1>
+    <visual>
+      <material>
+        <ambient>0 0 0 1</ambient>
+        <diffuse>0 0 0 1</diffuse>
+        <specular>0.1 0.1 0.1 1</specular>
+      </material>
+    </visual>
+    <!-- Black -->
   </gazebo>
   <!-- Caster Wheels -->
@@ -28,4 +55,12 @@
     <minDepth>0.001</minDepth>
     <maxVel>1.0</maxVel>
+    <visual>
+      <material>
+        <ambient>1 1 1 1</ambient>
+        <diffuse>1 1 1 1</diffuse>
+        <specular>0.1 0.1 0.1 1</specular>
+      </material>
+    </visual>
+    <!-- White -->
   </gazebo>
   <gazebo reference="caster_front_link">
@@ -36,4 +71,23 @@
     <minDepth>0.001</minDepth>
     <maxVel>1.0</maxVel>
+    <visual>
+      <material>
+        <ambient>1 1 1 1</ambient>
+        <diffuse>1 1 1 1</diffuse>
+        <specular>0.1 0.1 0.1 1</specular>
+      </material>
+    </visual>
+    <!-- White -->
   </gazebo>
+  <!-- Can -->
+  <!-- <gazebo reference="can_link">
+    <visual>
+      <material>
+        <ambient>1 0 0 1</ambient>
+        <diffuse>1 0 0 1</diffuse>
+        <specular>0.1 0.1 0.1 1</specular>
+      </material>
+    </visual>
+    (Red)
+  </gazebo> -->
 </robot>
