Commit message: Remove unnecessary .gitkeep files from various build directories

File: bumperbot_ws/install/bumperbot_description/share/bumperbot_description/urdf/bumperbot.urdf.xacro (robot description, xacro)
@@ -1 +1,210 @@
-/home/raz/projects/self_driving_OC_project/bumperbot_ws/src/bumperbot_description/urdf/bumperbot.urdf.xacro
+<?xml version="1.0"?>
+<robot name="bumperbot" xmlns:xacro="http://ros.org/wiki/xacro">
+  <!-- Start GZ or Ignition depending on ROS 2 Version -->
+  <xacro:arg name="is_ignition" default="True"/>
+  <!-- Determine between simulation and real hardware -->
+  <xacro:arg name="is_sim" default="True"/>
+  <!-- Include Common Properties -->
+  <xacro:include filename="$(find bumperbot_description)/urdf/common_properties.xacro" />
+  <!-- Include Gazebo Parameters -->
+  <xacro:include filename="$(find bumperbot_description)/urdf/bumperbot_gazebo.xacro" />
+  <!-- Include ros2_control Plugins -->
+  <xacro:include filename="$(find bumperbot_description)/urdf/bumperbot_ros2_control.xacro" />
+  <!-- Useful XACRO Variables (Properties) -->
+  <xacro:property name="effort" value="30.0" />
+  <xacro:property name="velocity" value="10.0" />
+  <!-- Dimensions -->
+  <xacro:property name="wheel_length" value="0.03" />
+  <xacro:property name="wheel_radius" value="0.033" />
+  <!-- Links -->
+  <link name="base_footprint"/>
+  <link name="base_link">
+    <visual>
+      <geometry>
+        <mesh filename="package://bumperbot_description/meshes/base_link.STL" />
+      </geometry>
+      <origin xyz="0 0 0" rpy="0 0 0" />
+      <material name="green" />
+    </visual>
+    <collision>
+      <geometry>
+        <mesh filename="package://bumperbot_description/meshes/base_link.STL" />
+      </geometry>
+      <origin xyz="0 0 0" rpy="0 0 0" />
+    </collision>
+    <inertial>
+      <origin xyz="0 0 0.04" rpy="0.0 0.25 0.3" />
+      <mass value="8.2573504e-01"/>
+      <inertia ixx="2.2124416e-02" ixy="-1.2294101e-04" ixz="3.4938785e-04"
+                                   iyy="2.1193702e-02"  iyz="-5.0120904e-05"
+                                                        izz="2.0064271e-02" />
+    </inertial>
+  </link>
+  <link name="wheel_right_link">
+    <visual>
+      <geometry>
+        <mesh filename="package://bumperbot_description/meshes/wheel_right_link.STL" />
+      </geometry>
+      <origin xyz="0 0 0" rpy="1.57 0 0" />
+      <material name="black" />
+    </visual>
+    <collision>
+      <geometry>
+        <sphere radius="${wheel_radius}"/>
+      </geometry>
+      <origin xyz="0 -${wheel_length / 2.0} 0" rpy="1.57 0 0" />
+    </collision>
+    <inertial>
+      <origin xyz="0 -0.014 0" rpy="0 0 0" />
+      <mass value="0.0530086090966721" />
+      <inertia ixx="1.88176298336665E-05" ixy="-4.8444933029987E-10" ixz="1.88163708851143E-08"
+                                          iyy="3.11510738647764E-05" iyz="-6.93560663069607E-11"
+                                                                     izz="1.8801969558182E-05" />
+    </inertial>
+  </link>
+  <link name="wheel_left_link">
+    <visual>
+      <geometry>
+        <mesh filename="package://bumperbot_description/meshes/wheel_left_link.STL" />
+      </geometry>
+      <origin xyz="0 0 0" rpy="-1.57 0 0" />
+      <material name="black" />
+    </visual>
+    <collision>
+      <geometry>
+        <sphere radius="${wheel_radius}"/>
+      </geometry>
+      <origin xyz="0 ${wheel_length / 2.0} 0" rpy="-1.57 0 0" />
+    </collision>
+    <inertial>
+      <origin xyz="0 0.014 0" rpy="0 0 0" />
+      <mass value="0.0530086043217644" />
+      <inertia ixx="1.8792911368909E-05"  ixy="3.31256392204584E-10" ixz="-1.14082001662767E-08"
+                                          iyy="3.11510738759073E-05" iyz="-3.60499245082192E-10"
+                                                                     izz="1.88266886146847E-05" />
+    </inertial>
+  </link>
+  <link name="caster_front_link">
+    <visual>
+      <geometry>
+        <mesh filename="package://bumperbot_description/meshes/caster_front_link.STL" />
+      </geometry>
+      <material name="white" />
+    </visual>
+      <origin xyz="0 0 0" rpy="0 0 0" />
+    <collision>
+      <geometry>
+        <sphere radius="0.005"/>
+      </geometry>
+      <origin xyz="0 0 0" rpy="0 0 0" />
+    </collision>
+    <inertial>
+      <origin xyz="3.89968128948481E-07 2.40073004698083E-07 0.00219173397061506" rpy="0 0 0" />
+      <mass value="1.44379265037903E-06" />
+      <inertia ixx="7.23075276010246E-11" ixy="-6.10956883467859E-16" ixz="2.22849693525031E-15"
+                                          iyy="3.8713793085917E-11"   iyz="2.93909858781952E-15"
+                                                                      izz="1.00967486676306E-10" />
+    </inertial>
+  </link>
+  <link name="caster_rear_link">
+    <visual>
+      <geometry>
+        <mesh filename="package://bumperbot_description/meshes/caster_rear_link.STL" />
+      </geometry>
+      <origin xyz="0 0 0" rpy="0 0 0" />
+      <material name="white" />
+    </visual>
+    <collision>
+      <geometry>
+        <sphere radius="0.005"/>
+      </geometry>
+      <origin xyz="0 0 0" rpy="0 0 0" />
+    </collision>
+    <inertial>
+      <origin xyz="3.8996812895542E-07 2.40073004698083E-07 0.00219173397061509" rpy="0 0 0" />
+      <mass value="1.44379265037902E-06" />
+      <inertia ixx="7.23075276010246E-11" ixy="-6.10956872363424E-16" ixz="2.22849693527207E-15"
+                                          iyy="3.87137930859167E-11"  iyz="2.939098587861E-15"
+                                                                      izz="1.00967486676306E-10" />
+    </inertial>
+  </link>
+  <link name="imu_link">
+    <visual>
+      <geometry>
+        <mesh filename="package://bumperbot_description/meshes/imu_link.STL" />
+      </geometry>
+      <origin xyz="0 0 0" rpy="0 0 0" />
+      <material name="white" />
+    </visual>
+    <collision>
+      <geometry>
+        <mesh filename="package://bumperbot_description/meshes/imu_link.STL" />
+      </geometry>
+      <origin xyz="0 0 0" rpy="0 0 0" />
+    </collision>
+    <inertial>
+      <origin xyz="-0.00552433659106688 0.000168210391520346 0.000514000497342681" rpy="0 0 0" />
+      <mass value="0.000528415362211671" />
+      <inertia ixx="1.46176048428261E-08" ixy="1.40015117949421E-10" ixz="-1.99633872937403E-12"
+                                          iyy="8.59662482954888E-09" iyz="7.52375112767959E-12"
+                                                                     izz="2.30279421279312E-08" />
+    </inertial>
+  </link>
+  <!-- <link name="can_link">
+    <visual>
+      <geometry>
+        <mesh filename="package://bumperbot_description/meshes/can.STL" />
+      </geometry>
+      <origin xyz="-0.0325 0.0325 0" rpy="1.57 0 0" />
+      <material name="red" />
+    </visual>
+    <collision>
+      <geometry>
+        <mesh filename="package://bumperbot_description/meshes/can.STL" />
+      </geometry>
+      <origin xyz="-0.0325 0.0325 0" rpy="1.57 0 0" />
+    </collision>
+  </link> -->
+  <!-- Joints -->
+  <joint name="base_joint" type="fixed">
+    <parent link="base_footprint"/>
+    <child link="base_link" />
+    <origin xyz="0 0 0.033" rpy="0 0 0"/>
+  </joint>
+  <joint name="wheel_right_joint" type="continuous">
+    <origin xyz="0 -0.0701101849418637 0" rpy="0 0 0" />
+    <parent link="base_link" />
+    <child link="wheel_right_link" />
+    <axis xyz="0 1 0" />
+  </joint>
+  <joint name="wheel_left_joint" type="continuous">
+    <origin xyz="0 0.0701101849418642 0" rpy="0 0 0" />
+    <parent link="base_link" />
+    <child link="wheel_left_link" />
+    <axis xyz="0 1 0" />
+  </joint>
+  <joint name="caster_front_joint" type="fixed">
+    <origin xyz="0.04755 0 -0.0275" rpy="0 0 0" />
+    <parent link="base_link" />
+    <child link="caster_front_link" />
+    <axis xyz="0 0 0" />
+  </joint>
+  <joint name="caster_rear_joint" type="fixed">
+    <origin xyz="-0.04755 0 -0.0275" rpy="0 0 0" />
+    <parent link="base_link" />
+    <child link="caster_rear_link" />
+    <axis xyz="0 0 0" />
+  </joint>
+  <joint name="imu_joint" type="fixed">
+    <origin xyz="0 0 0.0698986241758014" rpy="0 0 0" />
+    <parent link="base_link" />
+    <child link="imu_link" />
+    <axis xyz="0 0 0" />
+  </joint>
+  <!-- <joint name="can_joint" type="fixed">
+    <origin xyz="0 0 0.078" rpy="0 0 0" />
+    <parent link="base_link" />
+    <child link="can_link" />
+    <axis xyz="0 0 0" />
+  </joint> -->
+</robot>

File: bumperbot_ws/install/bumperbot_description/share/bumperbot_description/urdf/bumperbot_gazebo.xacro (robot description, xacro)
@@ -1 +1,165 @@
-/home/raz/projects/self_driving_OC_project/bumperbot_ws/src/bumperbot_description/urdf/bumperbot_gazebo.xacro
+<?xml version="1.0"?>
+<robot name="bumperbot" xmlns:xacro="http://ros.org/wiki/xacro">
+  <!-- Gazebo Plugin -->
+  <gazebo>
+    <!-- For ROS2 Humble -->
+    <xacro:if value="$(arg is_ignition)">
+      <plugin filename="ign_ros2_control-system" name="ign_ros2_control::IgnitionROS2ControlPlugin">
+        <parameters>$(find bumperbot_controller)/config/bumperbot_controllers.yaml</parameters>
+      </plugin>
+      <plugin filename="libignition-gazebo-imu-system.so" name="ignition::gazebo::systems::Imu">
+      </plugin>
+    </xacro:if>
+    <!-- For ROS2 Iron or above -->
+    <xacro:unless value="$(arg is_ignition)">
+      <plugin filename="gz_ros2_control-system" name="gz_ros2_control::GazeboSimROS2ControlPlugin">
+        <parameters>$(find bumperbot_controller)/config/bumperbot_controllers.yaml</parameters>
+      </plugin>
+      <plugin filename="gz-sim-imu-system" name="gazebo::sim::systems::Imu">
+      </plugin>
+    </xacro:unless>
+  </gazebo>
+  <gazebo reference="imu_link">
+    <sensor type="imu" name="imu">
+      <always_on>true</always_on>
+      <update_rate>100</update_rate>
+      <gz_frame_id>imu_link</gz_frame_id>
+      <topic>imu</topic>
+      <imu>
+        <angular_velocity>
+          <x>
+            <noise type="gaussian">
+              <mean>0.0</mean>
+              <stddev>2e-4</stddev>
+            </noise>
+          </x>
+          <y>
+            <noise type="gaussian">
+              <mean>0.0</mean>
+              <stddev>2e-4</stddev>
+            </noise>
+          </y>
+          <z>
+            <noise type="gaussian">
+              <mean>0.0</mean>
+              <stddev>2e-4</stddev>
+            </noise>
+          </z>
+        </angular_velocity>
+        <linear_acceleration>
+          <x>
+            <noise type="gaussian">
+              <mean>0.0</mean>
+              <stddev>1.7e-2</stddev>
+            </noise>
+          </x>
+          <y>
+            <noise type="gaussian">
+              <mean>0.0</mean>
+              <stddev>1.7e-2</stddev>
+            </noise>
+          </y>
+          <z>
+            <noise type="gaussian">
+              <mean>0.0</mean>
+              <stddev>1.7e-2</stddev>
+            </noise>
+          </z>
+        </linear_acceleration>
+      </imu>
+    </sensor>
+  </gazebo>
+  <!-- Base -->
+  <gazebo reference="base_link">
+    <visual>
+      <material>
+        <ambient>0 1 0 1</ambient>
+        <diffuse>0 1 0 1</diffuse>
+        <specular>0.1 0.1 0.1 1</specular>
+      </material>
+    </visual>
+    <!-- Green -->
+  </gazebo>
+  <!-- Wheels -->
+  <gazebo reference="wheel_left_link">
+    <mu1>1000000000000000.0</mu1>
+    <mu2>1000000000000000.0</mu2>
+    <kp>1000000000000.0</kp>
+    <kd>10.0</kd>
+    <minDepth>0.001</minDepth>
+    <maxVel>0.1</maxVel>
+    <fdir1>1 0 0</fdir1>
+    <visual>
+      <material>
+        <ambient>0 0 0 1</ambient>
+        <diffuse>0 0 0 1</diffuse>
+        <specular>0.1 0.1 0.1 1</specular>
+      </material>
+    </visual>
+    <!-- Black -->
+  </gazebo>
+  <gazebo reference="wheel_right_link">
+    <mu1>1000000000000000.0</mu1>
+    <mu2>1000000000000000.0</mu2>
+    <kp>1000000000000.0</kp>
+    <kd>10.0</kd>
+    <minDepth>0.001</minDepth>
+    <maxVel>0.1</maxVel>
+    <fdir1>1 0 0</fdir1>
+    <!-- Black -->
+    <visual>
+      <material>
+        <ambient>0 0 0 1</ambient>
+        <diffuse>0 0 0 1</diffuse>
+        <specular>0.1 0.1 0.1 1</specular>
+      </material>
+    </visual>
+    <!-- Black -->
+  </gazebo>
+  <!-- Caster Wheels -->
+  <gazebo reference="caster_rear_link">
+    <mu1>0.1</mu1>
+    <mu2>0.1</mu2>
+    <kp>1000000.0</kp>
+    <kd>100.0</kd>
+    <minDepth>0.001</minDepth>
+    <maxVel>1.0</maxVel>
+    <!-- White -->
+    <visual>
+      <material>
+        <ambient>1 1 1 1</ambient>
+        <diffuse>1 1 1 1</diffuse>
+        <specular>0.1 0.1 0.1 1</specular>
+      </material>
+    </visual>
+    <!-- White -->
+  </gazebo>
+  <gazebo reference="caster_front_link">
+    <mu1>0.1</mu1>
+    <mu2>0.1</mu2>
+    <kp>1000000.0</kp>
+    <kd>100.0</kd>
+    <minDepth>0.001</minDepth>
+    <maxVel>1.0</maxVel>
+    <!-- White -->
+    <visual>
+      <material>
+        <ambient>1 1 1 1</ambient>
+        <diffuse>1 1 1 1</diffuse>
+        <specular>0.1 0.1 0.1 1</specular>
+      </material>
+    </visual>
+    <!-- White -->
+  </gazebo>
+  <!-- Can -->
+  <!-- <gazebo reference="can_link">
+    <visual>
+      <material>
+        <ambient>1 0 0 1</ambient>
+        <diffuse>1 0 0 1</diffuse>
+        <specular>0.1 0.1 0.1 1</specular>
+      </material>
+    </visual>
+    (Red)
+  </gazebo> -->
+</robot>

File: bumperbot_ws/install/bumperbot_description/share/bumperbot_description/urdf/bumperbot_ros2_control.xacro (robot description, xacro)
@@ -1 +1,43 @@
-/home/raz/projects/self_driving_OC_project/bumperbot_ws/src/bumperbot_description/urdf/bumperbot_ros2_control.xacro
+<?xml version="1.0"?>
+<robot xmlns:xacro="http://www.ros.org/wiki/xacro" name="bumperbot">
+    <ros2_control name="RobotSystem" type="system">
+        <!-- ros2_control Gazebo -->
+        <xacro:if value="$(arg is_sim)">
+            <!-- ROS 2 Humble -->
+            <xacro:if value="$(arg is_ignition)">
+                <hardware>
+                    <plugin>ign_ros2_control/IgnitionSystem</plugin>
+                </hardware>
+            </xacro:if>
+            <!-- ROS 2 Iron or above -->
+            <xacro:unless value="$(arg is_ignition)">
+                <hardware>
+                    <plugin>gz_ros2_control/GazeboSimSystem</plugin>
+                </hardware>
+            </xacro:unless>
+        </xacro:if>
+        <xacro:unless value="$(arg is_sim)">
+            <hardware>
+                <plugin>bumperbot_firmware/bumperbot_interface</plugin>
+                <param name="port">/dev/ttyUSB0</param>
+            </hardware>
+        </xacro:unless>
+        <!-- ros2_control Command Interfaces -->
+        <joint name="wheel_right_joint">
+            <command_interface name="velocity">
+              <param name="min">-1</param>
+              <param name="max">1</param>
+            </command_interface>
+            <state_interface name="position" />
+            <state_interface name="velocity" />
+        </joint>
+        <joint name="wheel_left_joint">
+            <command_interface name="velocity">
+              <param name="min">-1</param>
+              <param name="max">1</param>
+            </command_interface>
+            <state_interface name="position" />
+            <state_interface name="velocity" />
+        </joint>
+    </ros2_control>
+</robot>

File: bumperbot_ws/install/bumperbot_description/share/bumperbot_description/urdf/common_properties.xacro (robot description, xacro)
@@ -1 +1,59 @@
-/home/raz/projects/self_driving_OC_project/bumperbot_ws/src/bumperbot_description/urdf/common_properties.xacro
+<?xml version="1.0"?>
+<robot xmlns:xacro="http://www.ros.org/wiki/xacro">
+    <!--                            Common Colors                            -->
+    <material name="red">
+        <color rgba="0.5 0 0 1" />
+    </material>
+    <material name="green">
+        <color rgba="0 0.5 0 1" />
+    </material>
+    <material name="blue">
+        <color rgba="0 0 0.5 1" />
+    </material>
+    <material name="grey">
+        <color rgba="0.5 0.5 0.5 1" />
+    </material>
+    <material name="orange">
+        <color rgba="1 0.65 0 1" />
+    </material>
+    <material name="yellow">
+        <color rgba="1 1 0 1" />
+    </material>
+    <material name="black">
+        <color rgba="0 0 0 1"/>
+    </material>
+    <material name="white">
+        <color rgba="1.0 1.0 1.0 1.0" />
+    </material>
+    <material name="transparent_black">
+        <color rgba="0 0 0 0.5"/>
+    </material>
+    <!--                     Common Momentum of Inertia                     -->
+    <xacro:macro name="box_inertia" params="m l w h xyz rpy">
+        <inertial>
+            <origin xyz="${xyz}" rpy="${rpy}" />
+            <mass value="${m}" />
+            <inertia ixx="${(m/12) * (h*h + l*l)}" ixy="0"                        ixz="0"
+                                                   iyy="${(m/12) * (w*w + l*l)}"  iyz="0"
+                                                                                  izz="${(m/12) * (w*w + h*h)}" />
+        </inertial>
+    </xacro:macro>
+    <xacro:macro name="cylinder_inertia" params="m r h xyz rpy">
+        <inertial>
+            <origin xyz="${xyz}" rpy="${rpy}" />
+            <mass value="${m}" />
+            <inertia ixx="${(1/12) * m * (3*r*r + h*h)}"  ixy="0"                              ixz="0"
+                                                          iyy="${(1/12) * m * (3*r*r + h*h)}"  iyz="0"
+                                                                                               izz="${(1/2) * m * (r*r)}" />
+        </inertial>
+    </xacro:macro>
+    <xacro:macro name="sphere_inertia" params="m r xyz rpy">
+        <inertial>
+            <origin xyz="${xyz}" rpy="${rpy}" />
+            <mass value="${m}" />
+            <inertia ixx="${(2/5) * m * (r*r)}"  ixy="0"                     ixz="0"
+                                                 iyy="${(2/5) * m * (r*r)}"  iyz="0"
+                                                                             izz="${(2/5) * m * (r*r)}" />
+        </inertial>
+    </xacro:macro>
+</robot>

File: bumperbot_ws/src/bumperbot_description/urdf/bumperbot.urdf.xacro (robot description, xacro)
@@ -3,4 +3,6 @@
   <!-- Start GZ or Ignition depending on ROS 2 Version -->
   <xacro:arg name="is_ignition" default="True"/>
+  <!-- Determine between simulation and real hardware -->
+  <xacro:arg name="is_sim" default="True"/>
   <!-- Include Common Properties -->
   <xacro:include filename="$(find bumperbot_description)/urdf/common_properties.xacro" />

File: bumperbot_ws/src/bumperbot_description/urdf/bumperbot_ros2_control.xacro (robot description, xacro)
@@ -3,14 +3,22 @@
     <ros2_control name="RobotSystem" type="system">
         <!-- ros2_control Gazebo -->
-        <!-- ROS 2 Humble -->
-        <xacro:if value="$(arg is_ignition)">
+        <xacro:if value="$(arg is_sim)">
+            <!-- ROS 2 Humble -->
+            <xacro:if value="$(arg is_ignition)">
+                <hardware>
+                    <plugin>ign_ros2_control/IgnitionSystem</plugin>
+                </hardware>
+            </xacro:if>
+            <!-- ROS 2 Iron or above -->
+            <xacro:unless value="$(arg is_ignition)">
+                <hardware>
+                    <plugin>gz_ros2_control/GazeboSimSystem</plugin>
+                </hardware>
+            </xacro:unless>
+        </xacro:if>
+        <xacro:unless value="$(arg is_sim)">
             <hardware>
-                <plugin>ign_ros2_control/IgnitionSystem</plugin>
-            </hardware>
-        </xacro:if>
-        <!-- ROS 2 Iron or above -->
-        <xacro:unless value="$(arg is_ignition)">
-            <hardware>
-                <plugin>gz_ros2_control/GazeboSimSystem</plugin>
+                <plugin>bumperbot_firmware/bumperbot_interface</plugin>
+                <param name="port">/dev/ttyUSB0</param>
             </hardware>
         </xacro:unless>
